Commit message: Add drone functionality and configuration files for Thaiquiri model
- Updated setup.py to include necessary launch files and scripts.
- Enhanced thaiquiri.urdf with additional sensors and devices.
- Created disparity_node.yaml for disparity configuration.
- Implemented bgra_to_bgr.py for image format conversion.
- Developed fix_camera_info.py to correct camera info messages.
- Added drone_launch.py for launching the drone simulation.
- Introduced .gitignore to exclude unnecessary files.

File: src/thaiquiri_webots/resource/thaiquiri.urdf (robot description, URDF)
Before this commit: robot /home/ubuntu/ros_ws/src/thaiquiri_webots/resource/thaiquiri.urdf, 21 links, 20 joints
Links:
- added link imu_livox
Joints:
- added joint lidar_livox_imu_livox_joint: type fixed, parent lidar_livox, child imu_livox, origin xyz=0 0 0 rpy=0 0 0
- joint ZED_X_Mini_camera_camera_left_joint: origin xyz=-0.025 0.003 0 rpy=-1.570796 0 -1.570796 -> xyz=-0.025 0.003 0 rpy=-0.523793 -1.570792 -1.047006
- joint ZED_X_Mini_camera_camera_right_joint: origin xyz=0.025 0.003 0.003 rpy=-1.570796 0 -1.570796 -> xyz=0.025 0.003 0.003 rpy=-0.523793 -1.570792 -1.047006

Commit message: Add sensors and update device references in Thaiquiri model

File: src/thaiquiri_webots/resource/thaiquiri.urdf (robot description, URDF)
Before this commit: robot thaiquiri, 22 links, 21 joints
Links:
- removed link imu_livox
- added link accelerometer_cube
- added link accelerometer_livox
- added link altimeter_cube
- added link compass_cube
- added link gyro_cube
- added link gyro_livox
Joints:
- removed joint lidar_livox_imu_livox_joint
- added joint cube_orange_accelerometer_cube_joint: type fixed, parent cube_orange, child accelerometer_cube, origin xyz=0 0 0 rpy=0 0 0
- added joint cube_orange_altimeter_cube_joint: type fixed, parent cube_orange, child altimeter_cube, origin xyz=0 0 0 rpy=0 0 0
- added joint cube_orange_compass_cube_joint: type fixed, parent cube_orange, child compass_cube, origin xyz=0 0 0 rpy=0 0 0
- added joint cube_orange_gyro_cube_joint: type fixed, parent cube_orange, child gyro_cube, origin xyz=0 0 0 rpy=0 0 0
- added joint lidar_livox_accelerometer_livox_joint: type fixed, parent lidar_livox, child accelerometer_livox, origin xyz=0 0 0 rpy=0 0 0
- added joint lidar_livox_gyro_livox_joint: type fixed, parent lidar_livox, child gyro_livox, origin xyz=0 0 0 rpy=0 0 0

Commit message: Update launch configuration and URDF for Thaiquiri model: enable RTAB-Map, adjust camera joint origins, and define base footprint link.

File: src/thaiquiri_webots/resource/thaiquiri.urdf (robot description, URDF)
Before this commit: robot thaiquiri, 27 links, 26 joints
Links:
- added link base_footprint
Joints:
- added joint base_footprint_to_base_link: type fixed, parent base_footprint, child base_link, origin xyz=0 0 0 rpy=1.5708 0 1.5708
- joint ZED_X_Mini_camera_camera_left_joint: origin xyz=-0.025 0.003 0 rpy=-0.523793 -1.570792 -1.047006 -> xyz=-0.025 0.003 0 rpy=0 0 0
- joint ZED_X_Mini_camera_camera_right_joint: origin xyz=0.025 0.003 0.003 rpy=-0.523793 -1.570792 -1.047006 -> xyz=0.025 0.003 0.003 rpy=0 0 0
